File: src/KiCad/MagicQuartz-Mega/MagicQuartz-Mega.kicad_pcb (KiCad board)
At the start: 2 copper layers, 82.6 x 50.2 mm, 33 parts, among them J1 Analog Out, J2 Power, J3 DC/DC, J4 Sensor, SW1 Left, SW2 Right, SW3 Down, SW4 Up, U1 MEGA 2560 PRO, U2 LM358

Commit message: Update to 1.04
Clarify voltages and update documentation
Parts:
- R4: value 0.15 / 5W -> 0.15 / 3W
- U1: value MEGA 2560 PRO -> MEGA_2560_PRO
Connections:
- net +12V renamed +7.5V
- net +28V renamed +24V
Other:
- board text added: "24V OUT"
- board text added: "7.5V IN"
- board text added: "PCB Rev. 1.04"
- board text removed: "12V IN"
- board text removed: "28V OUT"
- board text removed: "PCB Rev. 1.02"
